File: Hardware/node_sensor/_restore_backup_2026-05-22T14-22-20-146/node_sensor.kicad_sch (KiCad schematic)
At the start: 13 parts, among them J1 Solar_Pannel, U1 TPS63020, U2 INA219, U3 E32-433, U4 DevKitSTM32, U5 BMP-388, U6 SHT30, U7 BMS-1s

Commit message: completed v1 node sensor
Parts:
- C2, C3: footprint MY_FOOTPRINTS:C_0805 -> (none)
- J1: footprint MY_FOOTPRINTS:Conn_XH-P2.54mm-2P -> (none)
Connections:
- net GND: no longer U1.2 (GND), U7.4 (P-)
- net Pin+: now also J1.2 (Pin_2); no longer J1.1 (Pin_2)
- net Pin-: now also J1.1 (Pin_1); no longer J1.2 (Pin_1)
- new net: U1.2 (GND), U7.4 (P-)
Changed lines of the file:
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@@
 	(wire
 		(pts
-			(xy 62.23 64.77) (xy 62.23 66.04)
-		)
-		(stroke
-			(width 0)
-			(type default)
-		)
-	)
-	(wire
-		(pts
 			(xy 55.88 62.23) (xy 57.15 62.23)
 		)
@@
 	(wire
 		(pts
+			(xy 58.42 64.77) (xy 66.04 64.77)
+		)
+		(stroke
+			(width 0)
+			(type default)
+		)
+	)
+	(wire
+		(pts
 			(xy 67.31 34.29) (xy 67.31 35.56)
 		)
@@
 	(wire
 		(pts
-			(xy 66.04 64.77) (xy 62.23 64.77)
-		)
-		(stroke
-			(width 0)
-			(type default)
-		)
-	)
-	(wire
-		(pts
 			(xy 163.83 86.36) (xy 163.83 87.63)
 		)
@@
 	(wire
 		(pts
+			(xy 58.42 69.85) (xy 58.42 64.77)
+		)
+		(stroke
+			(width 0)
+			(type default)
+		)
+	)
+	(wire
+		(pts
 			(xy 163.83 72.39) (xy 167.64 72.39)
 		)
@@
 			)
 		)
-		(property "Footprint" "MY_FOOTPRINTS:C_0805"
+		(property "Footprint" ""
 			(at 55.88 31.75 0)
 			(hide yes)
@@
 			)
 		)
-		(property "Footprint" "MY_FOOTPRINTS:Conn_XH-P2.54mm-2P"
+		(property "Footprint" ""
 			(at 16.51 71.12 0)
 			(hide yes)
@@
 			)
 		)
-		(property "Footprint" "MY_FOOTPRINTS:C_0805"
+		(property "Footprint" ""
 			(at 67.31 31.75 0)
 			(hide yes)
@@
 	(symbol
 		(lib_id "power:GND")
-		(at 58.42 69.85 0)
-		(unit 1)
-		(body_style 1)
-		(exclude_from_sim no)
-		(in_bom yes)
-		(on_board yes)
-		(in_pos_files yes)
-		(dnp no)
-		(property "Reference" "#PWR015"
-			(at 58.42 76.2 0)
-			(hide yes)
-			(show_name no)
-			(do_not_autoplace no)
-			(effects
-				(font
-					(size 1.27 1.27)
-				)
-			)
-		)
-		(property "Value" "GND"
-			(at 59.944 73.66 0)
-			(show_name no)
-			(do_not_autoplace no)
-			(effects
-				(font
-					(size 1.27 1.27)
-				)
-			)
-		)
-		(property "Footprint" ""
-			(at 58.42 69.85 0)
-			(hide yes)
-			(show_name no)
-			(do_not_autoplace no)
-			(effects
-				(font
-					(size 1.27 1.27)
-				)
-			)
-		)
-		(property "Datasheet" ""
-			(at 58.42 69.85 0)
-			(hide yes)
-			(show_name no)
-			(do_not_autoplace no)
-			(effects
-				(font
-					(size 1.27 1.27)
-				)
-			)
-		)
-		(property "Description" "Power symbol creates a global label with name \"GND\" , ground"
-			(at 58.42 69.85 0)
-			(hide yes)
-			(show_name no)
-			(do_not_autoplace no)
-			(effects
-				(font
-					(size 1.27 1.27)
-				)
-			)
-		)
-		(pin "1"
-		)
-		(instances
-			(project "node_sensor"
-				(path "/9862bc29-5cf5-4b17-a93f-a6d59e2841b5"
-					(reference "#PWR015")
-					(unit 1)
-				)
-			)
-		)
-	)
-	(symbol
-		(lib_id "power:GND")
 		(at 163.83 64.77 270)
 		(unit 1)
@@
 					(unit 1)
 				)
-			)
-		)
-	)
-	(symbol
-		(lib_id "power:GND")
-		(at 62.23 66.04 270)
-		(unit 1)
-		(body_style 1)
-		(exclude_from_sim no)
-		(in_bom yes)
-		(on_board yes)
-		(in_pos_files yes)
-		(dnp no)
-		(property "Reference" "#PWR016"
-			(at 55.88 66.04 0)
-			(hide yes)
-			(show_name no)
-			(do_not_autoplace no)
-			(effects
-				(font
-					(size 1.27 1.27)
-				)
-			)
-		)
-		(property "Value" "GND"
-			(at 61.976 64.008 90)
-			(show_name no)
-			(do_not_autoplace no)
-			(effects
-				(font
-					(size 1.27 1.27)
-				)
-				(justify right)
-			)
-		)
-		(property "Footprint" ""
-			(at 62.23 66.04 0)
-			(hide yes)
-			(show_name no)
-			(do_not_autoplace no)
-			(effects
-				(font
-					(size 1.27 1.27)
-				)
-			)
-		)
-		(property "Datasheet" ""
-			(at 62.23 66.04 0)
-			(hide yes)
-			(show_name no)
-			(do_not_autoplace no)
-			(effects
-				(font
-					(size 1.27 1.27)
-				)
-			)
-		)
-		(property "Description" "Power symbol creates a global label with name \"GND\" , ground"
-			(at 62.23 66.04 0)
-			(hide yes)
-			(show_name no)
-			(do_not_autoplace no)
-			(effects
-				(font
-					(size 1.27 1.27)
-				)
-			)
-		)
-		(pin "1"
-		)
-		(instances
-			(project "node_sensor"
-				(path "/9862bc29-5cf5-4b17-a93f-a6d59e2841b5"
-					(reference "#PWR016")
-					(unit 1)
-				)
